Commit message: Limited joint Puma560

File: robots/puma560_description/urdf/puma560_robot.urdf (robot description, URDF)
Before this commit: robot Puma560, 7 links, 6 joints
Joints:
- joint j1: limit lower=-3.14159265 upper=3.14159265 effort=1000.0 velocity=0 -> lower=-2.793 upper=2.793 effort=1000.0 velocity=0
- joint j2: limit lower=-1.570796325 upper=1.570796325 effort=1000.0 velocity=0 -> lower=-2.182 upper=2.182 effort=1000.0 velocity=0
- joint j3: limit lower=-1.570796325 upper=1.570796325 effort=1000.0 velocity=0 -> lower=-2.356 upper=2.356 effort=1000.0 velocity=0
- joint j4: limit lower=-1.570796325 upper=1.570796325 effort=1000.0 velocity=0 -> lower=-2.443 upper=2.443 effort=1000.0 velocity=0
- joint j5: limit lower=-1.570796325 upper=1.570796325 effort=1000.0 velocity=0 -> lower=-1.745 upper=1.745 effort=1000.0 velocity=0
- joint j6: limit lower=-1.570796325 upper=1.570796325 effort=1000.0 velocity=0 -> lower=-4.643 upper=4.643 effort=1000.0 velocity=0

File: robots/puma560_description/urdf/puma560_robot.urdf.xacro (robot description, xacro)
@@ -50,5 +50,5 @@
     <origin xyz="0 0 ${d_1}" rpy="${M_PI/2} 0 0"/>
     <axis xyz="0 1 0"/> <!-- This is descibed in child frame -->
-    <limit effort="1000.0" lower="${-M_PI}" upper="${M_PI}" velocity="0"/>
+    <limit effort="1000.0" lower="${-M_PI*160/180}" upper="${M_PI*160/180}" velocity="0"/>
   </joint>
   <link name="link3">
@@ -66,5 +66,5 @@
     <origin xyz="0 0 0" rpy="0 0 0"/>
     <axis xyz="0 0 1"/> <!-- This is descibed in child frame -->
-    <limit effort="1000.0" lower="${-M_PI/2}" upper="${M_PI/2}" velocity="0"/>
+    <limit effort="1000.0" lower="${-M_PI*125/180}" upper="${M_PI*125/180}" velocity="0"/>
   </joint>
   <link name="link4">
@@ -82,5 +82,5 @@
     <origin xyz="${a_2} ${a_3} ${d_2}" rpy="0 0 ${-M_PI/2}"/>
     <axis xyz="0 0 1"/> <!-- This is descibed in child frame -->
-    <limit effort="1000.0" lower="${-M_PI/2}" upper="${M_PI/2}" velocity="0"/>
+    <limit effort="1000.0" lower="${-M_PI*135/180}" upper="${M_PI*135/180}" velocity="0"/>
   </joint>
   <link name="link5">
@@ -98,5 +98,5 @@
     <origin xyz="0 0 0" rpy="${M_PI/2} 0 ${M_PI/2}"/>
     <axis xyz="0 0 1"/>
-    <limit effort="1000.0" lower="${-M_PI/2}" upper="${M_PI/2}" velocity="0"/>
+    <limit effort="1000.0" lower="${-M_PI*140/180}" upper="${M_PI*140/180}" velocity="0"/>
   </joint>
   <link name="link6">
@@ -114,5 +114,5 @@
     <origin xyz="0 0 ${d_4}" rpy="${M_PI/2} 0 0"/>
     <axis xyz="0 0 1"/>
-    <limit effort="1000.0" lower="${-M_PI/2}" upper="${M_PI/2}" velocity="0"/>
+    <limit effort="1000.0" lower="${-M_PI*100/180}" upper="${M_PI*100/180}" velocity="0"/>
   </joint>
   <link name="link7">
@@ -130,5 +130,5 @@
     <origin xyz="0 ${d_6} 0" rpy="${-M_PI/2} 0 0"/>
     <axis xyz="0 0 1"/>
-    <limit effort="1000.0" lower="${-M_PI/2}" upper="${M_PI/2}" velocity="0"/>
+    <limit effort="1000.0" lower="${-M_PI*266/180}" upper="${M_PI*266/180}" velocity="0"/>
   </joint>
 </robot>
